File: base/mobile_robot.kicad_sch (KiCad schematic)
At the start: 74 parts, among them J1 USB_B_Micro, J2 Conn_02x05_Odd_Even, J3 Motor Power, J4 Conn_01x06, J5 Conn_01x06, Q1 BSS138, Q2 BSS138, Q3 BSS138, Q4 BSS138, SW1 SW_SPDT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

Commit message: Pretty much finished pcb layout and routing
Parts:
- added H1, H2, H3, H4: MountingHole, MountingHole:MountingHole_3.2mm_M3, symbol Mechanical:MountingHole
- SW1: footprint Button_Switch_THT:SW_E-Switch_EG1224_SPDT_Angled -> Button_Switch_SMD:SW_SPDT_PCM12
Connections:
- net HSE_IN: now also U2.5 (PD0); no longer U2.3 (PC14)
- net HSE_OUT: now also U2.6 (PD1); no longer U2.4 (PC15)
Other:
- note added: "Mounting holes"
Changed lines of the file:
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@@
   (no_connect (at 59.69 55.372))
   (no_connect (at 49.53 50.292))
-  (no_connect (at 126.238 58.42))
   (no_connect (at 159.258 83.82))
   (no_connect (at 159.258 88.9))
@@
   (no_connect (at 248.412 82.296))
   (no_connect (at 126.238 111.76))
-  (no_connect (at 126.238 60.96))
   (no_connect (at 159.258 81.28))
   (no_connect (at 126.238 114.3))
@@
   (no_connect (at 126.238 66.04))
   (no_connect (at 126.238 86.36))
+  (no_connect (at 126.238 68.58))
+  (no_connect (at 126.238 71.12))
   (wire (pts (xy 347.726 143.764) (xy 353.568 143.764))
     (stroke (width 0) (type default) (color 0 0 0 0))
@@
     (stroke (width 0) (type default) (color 0 0 0 0))
   )
-  (wire (pts (xy 122.428 68.58) (xy 126.238 68.58))
-    (stroke (width 0) (type default) (color 0 0 0 0))
-  )
   (wire (pts (xy 347.726 211.836) (xy 348.488 211.836))
     (stroke (width 0) (type default) (color 0 0 0 0))
   )
+  (polyline (pts (xy 195.58 126.746) (xy 195.58 157.226))
+    (stroke (width 0.5) (type solid) (color 0 0 0 0))
+  )
   (wire (pts (xy 41.275 32.512) (xy 41.275 35.687))
     (stroke (width 0) (type default) (color 0 0 0 0))
@@
     (stroke (width 0) (type default) (color 0 0 0 0))
   )
+  (polyline (pts (xy 195.58 126.746) (xy 272.796 126.746))
+    (stroke (width 0.5) (type solid) (color 0 0 0 0))
+  )
   (wire (pts (xy 369.951 82.55) (xy 369.951 81.534))
     (stroke (width 0) (type default) (color 0 0 0 0))
@@
     (stroke (width 0.5) (type solid) (color 0 0 0 0))
   )
-  (wire (pts (xy 122.428 71.12) (xy 126.238 71.12))
-    (stroke (width 0) (type default) (color 0 0 0 0))
-  )
   (wire (pts (xy 154.178 40.64) (xy 163.068 40.64))
     (stroke (width 0) (type default) (color 0 0 0 0))
@@
     (stroke (width 0) (type default) (color 0 0 0 0))
   )
+  (polyline (pts (xy 272.796 126.746) (xy 272.796 157.226))
+    (stroke (width 0.5) (type solid) (color 0 0 0 0))
+  )
   (wire (pts (xy 54.991 87.63) (xy 54.991 90.17))
     (stroke (width 0) (type default) (color 0 0 0 0))
@@
     (stroke (width 0) (type default) (color 0 0 0 0))
   )
+  (polyline (pts (xy 272.796 157.226) (xy 195.58 157.226))
+    (stroke (width 0.5) (type solid) (color 0 0 0 0))
+  )
   (wire (pts (xy 171.704 134.62) (xy 171.704 136.906))
     (stroke (width 0) (type default) (color 0 0 0 0))
@@
     (effects (font (size 2.54 2.54) (thickness 0.508) bold) (justify left bottom))
   )
+  (text "Mounting holes" (at 196.723 132.207 0)
+    (effects (font (size 2.54 2.54) (thickness 0.508) bold) (justify left bottom))
+  )
   (text "100nF per power pin, 10u bulk capacitor" (at 90.932 29.718 0)
     (effects (font (size 1.27 1.27)) (justify left bottom))
@@
     )
   )
-  (global_label "HSE_OUT" (shape input) (at 122.428 71.12 180) (fields_autoplaced)
+  (global_label "HSE_OUT" (shape input) (at 126.238 60.96 180) (fields_autoplaced)
     (effects (font (size 1.27 1.27)) (justify right))
-    (property "Intersheet References" "${INTERSHEET_REFS}" (id 0) (at 52.578 -1.27 0)
+    (property "Intersheet References" "${INTERSHEET_REFS}" (id 0) (at 56.388 -11.43 0)
       (effects (font (size 1.27 1.27)) hide)
     )
@@
     )
   )
-  (global_label "HSE_IN" (shape input) (at 122.428 68.58 180) (fields_autoplaced)
+  (global_label "HSE_IN" (shape input) (at 126.238 58.42 180) (fields_autoplaced)
     (effects (font (size 1.27 1.27)) (justify right))
-    (property "Intersheet References" "${INTERSHEET_REFS}" (id 0) (at 52.578 -1.27 0)
+    (property "Intersheet References" "${INTERSHEET_REFS}" (id 0) (at 56.388 -11.43 0)
       (effects (font (size 1.27 1.27)) hide)
     )
@@
     (pin "1")
   )
+  (symbol (lib_id "Mechanical:MountingHole") (at 218.821 139.446 0) (unit 1)
+    (in_bom yes) (on_board yes) (fields_autoplaced)
+    (property "Reference" "H1" (id 0) (at 222.25 138.1759 0)
+      (effects (font (size 1.27 1.27)) (justify left))
+    )
+    (property "Value" "MountingHole" (id 1) (at 222.25 140.7159 0)
+      (effects (font (size 1.27 1.27)) (justify left))
+    )
+    (property "Footprint" "MountingHole:MountingHole_3.2mm_M3" (id 2) (at 218.821 139.446 0)
+      (effects (font (size 1.27 1.27)) hide)
+    )
+    (property "Datasheet" "~" (id 3) (at 218.821 139.446 0)
+      (effects (font (size 1.27 1.27)) hide)
+    )
+  )
   (symbol (lib_id "Device:R_Small") (at 316.23 212.979 270) (unit 1)
     (in_bom yes) (on_board yes)
@@
     (pin "1")
   )
+  (symbol (lib_id "Mechanical:MountingHole") (at 241.046 147.955 0) (unit 1)
+    (in_bom yes) (on_board yes) (fields_autoplaced)
+    (property "Reference" "H4" (id 0) (at 243.713 146.6849 0)
+      (effects (font (size 1.27 1.27)) (justify left))
+    )
+    (property "Value" "MountingHole" (id 1) (at 243.713 149.2249 0)
+      (effects (font (size 1.27 1.27)) (justify left))
+    )
+    (property "Footprint" "MountingHole:MountingHole_3.2mm_M3" (id 2) (at 241.046 147.955 0)
+      (effects (font (size 1.27 1.27)) hide)
+    )
+    (property "Datasheet" "~" (id 3) (at 241.046 147.955 0)
+      (effects (font (size 1.27 1.27)) hide)
+    )
+  )
   (symbol (lib_id "Device:R_Small") (at 347.726 122.174 0) (unit 1)
     (in_bom yes) (on_board yes)
@@
     (property "Reference" "SW1" (id 0) (at 157.734 151.765 0))
     (property "Value" "SW_SPDT" (id 1) (at 157.734 161.925 0))
-    (property "Footprint" "Button_Switch_THT:SW_E-Switch_EG1224_SPDT_Angled" (id 2) (at 157.734 156.21 0)
+    (property "Footprint" "Button_Switch_SMD:SW_SPDT_PCM12" (id 2) (at 157.734 156.21 0)
       (effects (font (size 1.27 1.27)) hide)
     )
@@
     (pin "3")
   )
+  (symbol (lib_id "Mechanical:MountingHole") (at 218.948 148.209 0) (unit 1)
+    (in_bom yes) (on_board yes) (fields_autoplaced)
+    (property "Reference" "H3" (id 0) (at 222.25 146.9389 0)
+      (effects (font (size 1.27 1.27)) (justify left))
+    )
+    (property "Value" "MountingHole" (id 1) (at 222.25 149.4789 0)
+      (effects (font (size 1.27 1.27)) (justify left))
+    )
+    (property "Footprint" "MountingHole:MountingHole_3.2mm_M3" (id 2) (at 218.948 148.209 0)
+      (effects (font (size 1.27 1.27)) hide)
+    )
+    (property "Datasheet" "~" (id 3) (at 218.948 148.209 0)
+      (effects (font (size 1.27 1.27)) hide)
+    )
+  )
   (symbol (lib_id "power:PWR_FLAG") (at 163.068 33.02 0) (unit 1)
     (in_bom yes) (on_board yes) (fields_autoplaced)
@@
     (pin "1")
   )
+  (symbol (lib_id "Mechanical:MountingHole") (at 240.919 139.319 0) (unit 1)
+    (in_bom yes) (on_board yes) (fields_autoplaced)
+    (property "Reference" "H2" (id 0) (at 243.84 138.0489 0)
+      (effects (font (size 1.27 1.27)) (justify left))
+    )
+    (property "Value" "MountingHole" (id 1) (at 243.84 140.5889 0)
+      (effects (font (size 1.27 1.27)) (justify left))
+    )
+    (property "Footprint" "MountingHole:MountingHole_3.2mm_M3" (id 2) (at 240.919 139.319 0)
+      (effects (font (size 1.27 1.27)) hide)
+    )
+    (property "Datasheet" "~" (id 3) (at 240.919 139.319 0)
+      (effects (font (size 1.27 1.27)) hide)
+    )
+  )
   (symbol (lib_id "power:GND") (at 37.846 89.535 0) (unit 1)
     (in_bom yes) (on_board yes) (fields_autoplaced)
@@
       (reference "FB1") (unit 1) (value "120R") (footprint "Inductor_SMD:L_0603_1608Metric")
     )
+    (path "/37fb5a81-be9c-4778-a1a1-22aa968e390a"
+      (reference "H1") (unit 1) (value "MountingHole") (footprint "MountingHole:MountingHole_3.2mm_M3")
+    )
+    (path "/99bda189-f7be-49f9-81c7-1f618b950f9c"
+      (reference "H2") (unit 1) (value "MountingHole") (footprint "MountingHole:MountingHole_3.2mm_M3")
+    )
+    (path "/8df65b35-89f8-479f-b061-4fe678460196"
+      (reference "H3") (unit 1) (value "MountingHole") (footprint "MountingHole:MountingHole_3.2mm_M3")
+    )
+    (path "/48cc3411-7aa6-4fa5-9faa-88205e4e2f75"
+      (reference "H4") (unit 1) (value "MountingHole") (footprint "MountingHole:MountingHole_3.2mm_M3")
+    )
     (path "/b9313d61-0765-4bbe-8322-02f3de8db6cd"
       (reference "J1") (unit 1) (value "USB_B_Micro") (footprint "Connector_USB:USB_Micro-B_Molex_47346-0001")
@@
     )
     (path "/6c989432-ba20-498a-aeee-b0116b5b08f9"
-      (reference "SW1") (unit 1) (value "SW_SPDT") (footprint "Button_Switch_THT:SW_E-Switch_EG1224_SPDT_Angled")
+      (reference "SW1") (unit 1) (value "SW_SPDT") (footprint "Button_Switch_SMD:SW_SPDT_PCM12")
     )
     (path "/05b8381a-8a83-4eb2-a86d-9f15ed62725a"

Commit message: Finished PCB
Parts:
- J3: value Motor Power -> AMASS XT60PW
- U4: value L298HN -> L298N
Changed lines of the file:
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@@
       (effects (font (size 1.27 1.27)) (justify left))
     )
-    (property "Value" "L298HN" (id 1) (at 319.913 83.058 0)
+    (property "Value" "L298N" (id 1) (at 319.913 83.058 0)
       (effects (font (size 1.27 1.27)) (justify left))
     )
@@
     (in_bom yes) (on_board yes)
     (property "Reference" "J3" (id 0) (at 344.17 30.226 0))
-    (property "Value" "Motor Power" (id 1) (at 344.17 38.354 0))
+    (property "Value" "AMASS XT60PW" (id 1) (at 342.392 38.354 0))
     (property "Footprint" "Connector_AMASS:AMASS_XT60PW-M" (id 2) (at 344.17 35.56 0)
       (effects (font (size 1.27 1.27)) hide)
@@
     )
     (path "/b6955664-2ce3-4f83-9c6d-dc28d966ef71"
-      (reference "J3") (unit 1) (value "Motor Power") (footprint "Connector_AMASS:AMASS_XT60PW-M")
+      (reference "J3") (unit 1) (value "AMASS XT60PW") (footprint "Connector_AMASS:AMASS_XT60PW-M")
     )
     (path "/cbe1ab7d-4e0c-4855-ae81-c83b98288cb5"
@@
     )
     (path "/8a7323b1-0518-441d-ad43-c25c2f1e751d"
-      (reference "U4") (unit 1) (value "L298HN") (footprint "Package_TO_SOT_THT:TO-220-15_P2.54x2.54mm_StaggerOdd_Lead4.58mm_Vertical")
+      (reference "U4") (unit 1) (value "L298N") (footprint "Package_TO_SOT_THT:TO-220-15_P2.54x2.54mm_StaggerOdd_Lead4.58mm_Vertical")
     )
     (path "/b9dc75f3-e8e4-4a46-9b6e-c33865328879"
